File: examples/spice-parser/kicad-pyspice-example/kicad-pyspice-example.sch (KiCad schematic (older format))
At the start: 7 parts, among them X1 JackIn, X2 PowerIn, X3 Opamp, X4 JackOut

Commit message: KiCAD example project update
Parts:
- X3: symbol LM193 -> LM193-RESCUE-kicad-pyspice-example
Changed lines of the file:
@@
 $EndDescr
 $Comp
-L LM193 X3
+L LM193-RESCUE-kicad-pyspice-example X3
 U 1 1 55381082
 P 5450 3750
@@
 	4850 4200 4850 3850
 Wire Wire Line
-	4700 3850 4850 3850
-Wire Wire Line
-	4850 3850 4950 3850
+	4700 3850 4950 3850
 Connection ~ 4850 3850
 Wire Wire Line
@@
 Connection ~ 6350 3750
 Wire Wire Line
-	3950 4750 4750 4750
-Wire Wire Line
-	4750 4750 6550 4750
-Wire Wire Line
-	6550 4750 6750 4750
+	3950 4750 6750 4750
 Wire Wire Line
 	4950 3650 4750 3650
 Wire Wire Line
-	4750 3650 4750 4750
-Wire Wire Line
-	4750 4750 4750 4900
+	4750 3650 4750 4900
 Connection ~ 4750 4750
 $Comp
@@
 	4200 3100 4200 3300
 Wire Wire Line
-	5950 3750 6350 3750
-Wire Wire Line
-	6350 3750 6850 3750
+	5950 3750 6850 3750
 Wire Wire Line
 	6850 3850 6550 3850
@@
 	3600 3750 3950 3750
 Wire Wire Line
-	3950 3600 3950 3750
-Wire Wire Line
-	3950 3750 3950 4750
+	3950 3600 3950 4750
 Wire Wire Line
 	3600 3600 3950 3600
